Commit message: chore: Update launch file and URDF for spawing Robot

File: urdf/voice_controlled_robot.urdf (robot description, URDF)
Before this commit: robot test_robot, 2 links, 1 joints
Links:
- link base_link: mass None -> 1.0
- link body_link: mass None -> 1.0; geometry collision box size=0.3 0.3 0.2; visual box size=0.3 0.3 0.2

Commit message: chore: Update diff_drive_controller.yaml configuration file and voice_controlled_robot_gazebo.launch file

File: urdf/voice_controlled_robot.urdf (robot description, URDF)
Before this commit: robot test_robot, 2 links, 1 joints
Links:
- added link left_wheel; visual cylinder length=0.02 radius=0.05
- added link right_wheel; visual cylinder length=0.02 radius=0.05
Joints:
- added joint left_wheel_joint: type continuous, parent base_link, child left_wheel, origin xyz=0 0.15 0 rpy=0 0 0, axis 0 0 1
- added joint right_wheel_joint: type continuous, parent base_link, child right_wheel, origin xyz=0 -0.15 0 rpy=0 0 0, axis 0 0 1
